File: Watersphere mobo.kicad_sch (KiCad schematic)
At the start: 0 parts

Commit message: Motor Controller tings
Other:
- added sheet Motor Controller (untitled.kicad_sch)
Changed lines of the file:
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@@
+    )
+  )
+  (sheet (at 119.38 45.72) (size 39.37 20.32) (fields_autoplaced)
+    (stroke (width 0.1524) (type solid))
+    (fill (color 0 0 0 0.0000))
+    (property "Sheetname" "Motor Controller" (at 119.38 45.0084 0)
+      (effects (font (size 1.27 1.27)) (justify left bottom))
+    )
+    (property "Sheetfile" "untitled.kicad_sch" (at 119.38 66.6246 0)
+      (effects (font (size 1.27 1.27)) (justify left top))
+    )
+    (instances
+      (project "Watersphere mobo"
+        (path "/c4a63ad0-0af5-4f61-bde7-7fb53fc8413c" (page "5"))
+      )
     )
   )
