File: mcu.kicad_sch (KiCad schematic)
At the start: 0 parts

Commit message: Lotta stuff added
Parts:
- added C16: 10 uF, symbol Device:C
- added C17: 4.7 uF, symbol Device:C
- added C18: 1 uF, symbol Device:C
- added U7: ADA3708, ADA3708:MODULE_ADA3708, symbol Raspberry Pi Zero:ADA3708
Connections:
- new net +5v: C16.1, C17.1, C18.1, U7.4 (5V_2)
- new net GND: C16.2, C17.2, C18.2, U7.14 (GND_4), U7.20 (GND_5), U7.25 (GND_2), U7.30 (GND_6), U7.34 (GND_7), U7.39 (GND_3), U7.9 (GND_1)
- new net I2C_Bus1_SCL: U7.5 (GPIO3_SCL)
- new net I2C_Bus1_SDA: U7.3 (GPIO2_SDA)
Other:
- note added: "MCU Decoupling"

Commit message: Motor Controller tings
Connections:
- net PWM_Expander_CLK: now reaches U7.32 (GPIO12)
Changed lines of the file:
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@@
+    (stroke (width 0) (type default))
+  )
+  (wire (pts (xy 201.93 106.68) (xy 177.8 106.68))
     (stroke (width 0) (type default))
   )
@@
       (effects (font (size 1.27 1.27)) (justify left) hide)
     )
+  )
+  (global_label "PWM_Expander_CLK" (shape input) (at 201.93 106.68 0) (fields_autoplaced)
+    (effects (font (size 1.27 1.27)) (justify left))
+    (property "Intersheetrefs" "${INTERSHEET_REFS}" (at 223.1598 106.68 0)
+      (effects (font (size 1.27 1.27)) (justify left) hide)
+    )

Commit message: routing
Parts:
- C16, C17, C18: footprint (none) -> Capacitor_SMD:C_0603_1608Metric_Pad1.08x0.95mm_HandSolder
Connections:
- net BNO_Data_Ready: now reaches U7.13 (GPIO27_GEN2)
- net BNO_BOOTN: now reaches U7.15 (GPIO22_GEN3)
Changed lines of the file:
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@@
+    (stroke (width 0) (type default))
+  )
+  (wire (pts (xy 118.11 83.82) (xy 127 83.82))
     (stroke (width 0) (type default))
   )
@@
   )
   (wire (pts (xy 115.57 73.66) (xy 127 73.66))
+    (stroke (width 0) (type default))
+  )
+  (wire (pts (xy 118.11 86.36) (xy 127 86.36))
     (stroke (width 0) (type default))
   )
@@
     )
   )
+  (global_label "BNO_Data_Ready" (shape input) (at 118.11 83.82 180) (fields_autoplaced)
+    (effects (font (size 1.27 1.27)) (justify right))
+    (property "Intersheetrefs" "${INTERSHEET_REFS}" (at 99.4201 83.82 0)
+      (effects (font (size 1.27 1.27)) (justify right) hide)
+    )
+  )
   (global_label "+5v" (shape input) (at 69.85 25.4 0) (fields_autoplaced)
     (effects (font (size 1.27 1.27)) (justify left))
@@
     (effects (font (size 1.27 1.27)) (justify right))
     (property "Intersheetrefs" "${INTERSHEET_REFS}" (at 99.4805 73.66 0)
+      (effects (font (size 1.27 1.27)) (justify right) hide)
+    )
+  )
+  (global_label "BNO_BOOTN" (shape input) (at 118.11 86.36 180) (fields_autoplaced)
+    (effects (font (size 1.27 1.27)) (justify right))
+    (property "Intersheetrefs" "${INTERSHEET_REFS}" (at 104.0765 86.36 0)
       (effects (font (size 1.27 1.27)) (justify right) hide)
     )
@@
       (effects (font (size 1.27 1.27)) (justify left))
     )
-    (property "Footprint" "" (at 36.5252 33.02 0)
+    (property "Footprint" "Capacitor_SMD:C_0603_1608Metric_Pad1.08x0.95mm_HandSolder" (at 36.5252 33.02 0)
       (effects (font (size 1.27 1.27)) hide)
     )
@@
       (effects (font (size 1.27 1.27)) (justify left))
     )
-    (property "Footprint" "" (at 49.2252 33.02 0)
+    (property "Footprint" "Capacitor_SMD:C_0603_1608Metric_Pad1.08x0.95mm_HandSolder" (at 49.2252 33.02 0)
       (effects (font (size 1.27 1.27)) hide)
     )
@@
       (effects (font (size 1.27 1.27)) (justify left))
     )
-    (property "Footprint" "" (at 60.6552 33.02 0)
-      (effects (font (size 1.27 1.27)) hide)
-    )
+    (property "Footprint" "Capacitor_SMD:C_0603_1608Metric_Pad1.08x0.95mm_HandSolder" (at 60.6552 33.02 0)
+      (effects (font (size 1.27 1.27)) hide)
+    )

Commit message: Routing begin
Parts:
- removed C16: 10 uF, Capacitor_SMD:C_0603_1608Metric_Pad1.08x0.95mm_HandSolder, symbol Device:C
- removed C17: 4.7 uF, Capacitor_SMD:C_0603_1608Metric_Pad1.08x0.95mm_HandSolder, symbol Device:C
- removed C18: 1 uF, Capacitor_SMD:C_0603_1608Metric_Pad1.08x0.95mm_HandSolder, symbol Device:C
Connections:
- net +5v renamed Rasp_Vsupply
Other:
- note removed: "MCU Decoupling"
Changed lines of the file:
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@@
 (kicad_sch (version 20230121) (generator eeschema)
   (paper "A4")
-  (junction (at 35.56 25.4) (diameter 0) (color 0 0 0 0)
-  )
-  (junction (at 59.69 25.4) (diameter 0) (color 0 0 0 0)
-  )
-  (junction (at 48.26 25.4) (diameter 0) (color 0 0 0 0)
-  )
   (wire (pts (xy 187.96 109.22) (xy 177.8 109.22))
     (stroke (width 0) (type default))
   )
-  (wire (pts (xy 31.75 25.4) (xy 35.56 25.4))
-    (stroke (width 0) (type default))
-  )
   (wire (pts (xy 116.84 116.84) (xy 127 116.84))
     (stroke (width 0) (type default))
   )
-  (wire (pts (xy 59.69 25.4) (xy 69.85 25.4))
-    (stroke (width 0) (type default))
-  )
-  (wire (pts (xy 35.56 25.4) (xy 48.26 25.4))
-    (stroke (width 0) (type default))
-  )
   (wire (pts (xy 187.96 91.44) (xy 177.8 91.44))
     (stroke (width 0) (type default))
@@
     (stroke (width 0) (type default))
   )
-  (wire (pts (xy 48.26 25.4) (xy 59.69 25.4))
-    (stroke (width 0) (type default))
-  )
   (wire (pts (xy 187.96 104.14) (xy 177.8 104.14))
     (stroke (width 0) (type default))
@@
     (stroke (width 0) (type default))
   )
-  (wire (pts (xy 59.69 33.02) (xy 59.69 34.29))
-    (stroke (width 0) (type default))
-  )
   (wire (pts (xy 187.96 83.82) (xy 177.8 83.82))
     (stroke (width 0) (type default))
   )
-  (wire (pts (xy 35.56 33.02) (xy 35.56 34.29))
-    (stroke (width 0) (type default))
-  )
   (wire (pts (xy 116.84 99.06) (xy 127 99.06))
     (stroke (width 0) (type default))
@@
     (stroke (width 0) (type default))
   )
-  (wire (pts (xy 48.26 33.02) (xy 48.26 34.29))
-    (stroke (width 0) (type default))
-  )
   (rectangle (start 15.24 13.97) (end 87.63 43.18)
     (stroke (width 0) (type default))
     (fill (type none))
   )
-  (text "MCU Decoupling" (at 16.51 20.32 0)
-    (effects (font (size 4 4)) (justify left bottom))
-  )
   (global_label "I2C_Bus1_SDA" (shape input) (at 115.57 71.12 180) (fields_autoplaced)
     (effects (font (size 1.27 1.27)) (justify right))
     (property "Intersheetrefs" "${INTERSHEET_REFS}" (at 99.42 71.12 0)
-      (effects (font (size 1.27 1.27)) (justify right) hide)
-    )
-  )
-  (global_label "Rasp_Vsupply" (shape input) (at 31.75 25.4 180) (fields_autoplaced)
-    (effects (font (size 1.27 1.27)) (justify right))
-    (property "Intersheetrefs" "${INTERSHEET_REFS}" (at 16.084 25.4 0)
       (effects (font (size 1.27 1.27)) (justify right) hide)
     )
@@
     )
   )
-  (global_label "+5v" (shape input) (at 69.85 25.4 0) (fields_autoplaced)
-    (effects (font (size 1.27 1.27)) (justify left))
-    (property "Intersheetrefs" "${INTERSHEET_REFS}" (at 76.5053 25.4 0)
-      (effects (font (size 1.27 1.27)) (justify left) hide)
-    )
-  )
   (global_label "PWM_Expander_CLK" (shape input) (at 201.93 106.68 0) (fields_autoplaced)
     (effects (font (size 1.27 1.27)) (justify left))
@@
         (path "/c4a63ad0-0af5-4f61-bde7-7fb53fc8413c/3f8884fe-4665-4fba-a6c0-e9032b67a8f5"
           (reference "#PWR049") (unit 1)
-        )
-      )
-    )
-  )
-  (symbol (lib_id "power:GND") (at 59.69 34.29 0) (unit 1)
-    (in_bom yes) (on_board yes) (dnp no) (fields_autoplaced)
-    (property "Reference" "#PWR045" (at 59.69 40.64 0)
-      (effects (font (size 1.27 1.27)) hide)
-    )
-    (property "Value" "GND" (at 59.69 39.37 0)
-      (effects (font (size 1.27 1.27)))
-    )
-    (property "Footprint" "" (at 59.69 34.29 0)
-      (effects (font (size 1.27 1.27)) hide)
-    )
-    (property "Datasheet" "" (at 59.69 34.29 0)
-      (effects (font (size 1.27 1.27)) hide)
-    )
-    (pin "1")
-    (instances
-      (project "Watersphere mobo"
-        (path "/c4a63ad0-0af5-4f61-bde7-7fb53fc8413c/3f8884fe-4665-4fba-a6c0-e9032b67a8f5"
-          (reference "#PWR045") (unit 1)
         )
       )
@@
     )
   )
-  (symbol (lib_id "power:GND") (at 35.56 34.29 0) (unit 1)
-    (in_bom yes) (on_board yes) (dnp no) (fields_autoplaced)
-    (property "Reference" "#PWR043" (at 35.56 40.64 0)
-      (effects (font (size 1.27 1.27)) hide)
-    )
-    (property "Value" "GND" (at 35.56 39.37 0)
-      (effects (font (size 1.27 1.27)))
-    )
-    (property "Footprint" "" (at 35.56 34.29 0)
-      (effects (font (size 1.27 1.27)) hide)
-    )
-    (property "Datasheet" "" (at 35.56 34.29 0)
-      (effects (font (size 1.27 1.27)) hide)
-    )
-    (pin "1")
-    (instances
-      (project "Watersphere mobo"
-        (path "/c4a63ad0-0af5-4f61-bde7-7fb53fc8413c/3f8884fe-4665-4fba-a6c0-e9032b67a8f5"
-          (reference "#PWR043") (unit 1)
-        )
-      )
-    )
-  )
   (symbol (lib_id "power:GND") (at 187.96 83.82 0) (unit 1)
     (in_bom yes) (on_board yes) (dnp no) (fields_autoplaced)
@@
     )
   )
-  (symbol (lib_id "Device:C") (at 35.56 29.21 0) (unit 1)
-    (in_bom yes) (on_board yes) (dnp no)
-    (property "Reference" "C16" (at 38.1 27.94 0)
-      (effects (font (size 1.27 1.27)) (justify left))
-    )
-    (property "Value" "10 uF" (at 38.1 30.48 0)
-      (effects (font (size 1.27 1.27)) (justify left))
-    )
-    (property "Footprint" "Capacitor_SMD:C_0603_1608Metric_Pad1.08x0.95mm_HandSolder" (at 36.5252 33.02 0)
-      (effects (font (size 1.27 1.27)) hide)
-    )
-    (property "Datasheet" "~" (at 35.56 29.21 0)
-      (effects (font (size 1.27 1.27)) hide)
-    )
-    (pin "1")
-    (pin "2")
-    (instances
-      (project "Watersphere mobo"
-        (path "/c4a63ad0-0af5-4f61-bde7-7fb53fc8413c/3f8884fe-4665-4fba-a6c0-e9032b67a8f5"
-          (reference "C16") (unit 1)
-        )
-      )
-    )
-  )
-  (symbol (lib_id "Device:C") (at 48.26 29.21 0) (unit 1)
-    (in_bom yes) (on_board yes) (dnp no)
-    (property "Reference" "C17" (at 50.8 27.94 0)
-      (effects (font (size 1.27 1.27)) (justify left))
-    )
-    (property "Value" "4.7 uF" (at 50.8 30.48 0)
-      (effects (font (size 1.27 1.27)) (justify left))
-    )
-    (property "Footprint" "Capacitor_SMD:C_0603_1608Metric_Pad1.08x0.95mm_HandSolder" (at 49.2252 33.02 0)
-      (effects (font (size 1.27 1.27)) hide)
-    )
-    (property "Datasheet" "~" (at 48.26 29.21 0)
-      (effects (font (size 1.27 1.27)) hide)
-    )
-    (pin "1")
-    (pin "2")
-    (instances
-      (project "Watersphere mobo"
-        (path "/c4a63ad0-0af5-4f61-bde7-7fb53fc8413c/3f8884fe-4665-4fba-a6c0-e9032b67a8f5"
-          (reference "C17") (unit 1)
-        )
-      )
-    )
-  )
   (symbol (lib_id "power:GND") (at 187.96 109.22 0) (unit 1)
     (in_bom yes) (on_board yes) (dnp no) (fields_autoplaced)
@@
     )
   )
-  (symbol (lib_id "power:GND") (at 48.26 34.29 0) (unit 1)
-    (in_bom yes) (on_board yes) (dnp no) (fields_autoplaced)
-    (property "Reference" "#PWR044" (at 48.26 40.64 0)
-      (effects (font (size 1.27 1.27)) hide)
-    )
-    (property "Value" "GND" (at 48.26 39.37 0)
-      (effects (font (size 1.27 1.27)))
-    )
-    (property "Footprint" "" (at 48.26 34.29 0)
-      (effects (font (size 1.27 1.27)) hide)
-    )
-    (property "Datasheet" "" (at 48.26 34.29 0)
-      (effects (font (size 1.27 1.27)) hide)
-    )
-    (pin "1")
-    (instances
-      (project "Watersphere mobo"
-        (path "/c4a63ad0-0af5-4f61-bde7-7fb53fc8413c/3f8884fe-4665-4fba-a6c0-e9032b67a8f5"
-          (reference "#PWR044") (unit 1)
-        )
-      )
-    )
-  )
   (symbol (lib_id "power:GND") (at 116.84 116.84 0) (unit 1)
     (in_bom yes) (on_board yes) (dnp no) (fields_autoplaced)
@@
         )
       )
-    )
-  )
-  (symbol (lib_id "Device:C") (at 59.69 29.21 0) (unit 1)
-    (in_bom yes) (on_board yes) (dnp no)
-    (property "Reference" "C18" (at 62.23 27.94 0)
-      (effects (font (size 1.27 1.27)) (justify left))
-    )
-    (property "Value" "1 uF" (at 62.23 30.48 0)
-      (effects (font (size 1.27 1.27)) (justify left))
-    )
-    (property "Footprint" "Capacitor_SMD:C_0603_1608Metric_Pad1.08x0.95mm_HandSolder" (at 60.6552 33.02 0)
-      (effects (font (size 1.27 1.27)) hide)
-    )
-    (property "Datasheet" "~" (at 59.69 29.21 0)
-      (effects (font (size 1.27 1.27)) hide)
-    )
-    (pin "1")
-    (pin "2")
-    (instances
-      (project "Watersphere mobo"
-        (path "/c4a63ad0-0af5-4f61-bde7-7fb53fc8413c/3f8884fe-4665-4fba-a6c0-e9032b67a8f5"
-          (reference "C18") (unit 1)
-        )
-      )

Commit message: gps started
Parts:
- added U9: TESEO-LIV3R, ARRAY_LIV3R_STM, symbol Teseo Liver:TESEO-LIV3R
Connections:
- net I2C_Bus1_SCL: now also U9.17 (SCL)
- net I2C_Bus1_SDA: now also U9.16 (SDA)
- no-connect marks 0 -> 6
Changed lines of the file:
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@@
 (kicad_sch (version 20230121) (generator eeschema)
   (paper "A4")
+  (no_connect (at 118.11 140.97))
+  (no_connect (at 118.11 143.51))
+  (no_connect (at 118.11 146.05))
+  (no_connect (at 173.99 146.05))
+  (no_connect (at 173.99 138.43))
+  (no_connect (at 118.11 148.59))
   (wire (pts (xy 187.96 109.22) (xy 177.8 109.22))
     (stroke (width 0) (type default))
   )
+  (wire (pts (xy 179.07 143.51) (xy 173.99 143.51))
+    (stroke (width 0) (type default))
+  )
   (wire (pts (xy 116.84 116.84) (xy 127 116.84))
+    (stroke (width 0) (type default))
+  )
+  (wire (pts (xy 179.07 140.97) (xy 173.99 140.97))
     (stroke (width 0) (type default))
   )
@@
     (effects (font (size 1.27 1.27)) (justify left))
     (property "Intersheetrefs" "${INTERSHEET_REFS}" (at 223.1598 106.68 0)
+      (effects (font (size 1.27 1.27)) (justify left) hide)
+    )
+  )
+  (global_label "I2C_Bus1_SDA" (shape input) (at 179.07 143.51 0) (fields_autoplaced)
+    (effects (font (size 1.27 1.27)) (justify left))
+    (property "Intersheetrefs" "${INTERSHEET_REFS}" (at 195.22 143.51 0)
+      (effects (font (size 1.27 1.27)) (justify left) hide)
+    )
+  )
+  (global_label "I2C_Bus1_SCL" (shape input) (at 179.07 140.97 0) (fields_autoplaced)
+    (effects (font (size 1.27 1.27)) (justify left))
+    (property "Intersheetrefs" "${INTERSHEET_REFS}" (at 195.1595 140.97 0)
       (effects (font (size 1.27 1.27)) (justify left) hide)
     )
@@
         )
       )
+    )
+  )
+  (symbol (lib_id "Teseo Liver:TESEO-LIV3R") (at 118.11 138.43 0) (unit 1)
+    (in_bom yes) (on_board yes) (dnp no) (fields_autoplaced)
+    (property "Reference" "U9" (at 146.05 128.27 0)
+      (effects (font (size 1.524 1.524)))
+    )
+    (property "Value" "TESEO-LIV3R" (at 146.05 130.81 0)
+      (effects (font (size 1.524 1.524)))
+    )
+    (property "Footprint" "ARRAY_LIV3R_STM" (at 118.11 138.43 0)
+      (effects (font (size 1.27 1.27) italic) hide)
+    )
+    (property "Datasheet" "TESEO-LIV3R" (at 118.11 138.43 0)
+      (effects (font (size 1.27 1.27) italic) hide)
+    )
+    (pin "1")
+    (pin "10")
+    (pin "11")
+    (pin "12")
+    (pin "13")
+    (pin "14")
+    (pin "15")
+    (pin "16")
+    (pin "17")
+    (pin "18")
+    (pin "2")
+    (pin "3")
+    (pin "4")
+    (pin "5")
+    (pin "6")
+    (pin "7")
+    (pin "8")
+    (pin "9")
+    (instances
+      (project "Watersphere mobo"
+        (path "/c4a63ad0-0af5-4f61-bde7-7fb53fc8413c/3f8884fe-4665-4fba-a6c0-e9032b67a8f5"
+          (reference "U9") (unit 1)
+        )
+      )

Commit message: Tedi Check dis over pls.
Parts:
- added C4: 100nF, Capacitor_SMD:C_0603_1608Metric_Pad1.08x0.95mm_HandSolder, symbol Device:C
- added C4: 10 uF, Capacitor_SMD:C_0603_1608Metric_Pad1.08x0.95mm_HandSolder, symbol Device:C
- added U10: 734120114, UFL:73412-0114_MOL, symbol UFL:734120114
- U9: footprint ARRAY_LIV3R_STM -> Teseo Liv3r:ARRAY_LIV3R_STM
Connections:
- net GND: now also U9.1 (GND), U9.10 (GND_RF), U9.12 (GND_RF), C4.2, C4.2, U10.2 (GROUND), U10.3 (GROUND), U10.4 (GROUND)
- net Solenoid_Driver: now reaches U7.29 (GPIO5)
- net at U9.11 (RF_IN): now also U10.1 (SIGNAL)
- net +3.3V: now reaches U9.6 (VBATT)
- net +3.3V: now also U9.7 (VCC_IO), U9.8 (VCC), C4.1, C4.1
- no-connect marks 6 -> 9
