File: Watersphere mobo.kicad_pcb (KiCad board)
At the start: 4 copper layers, 74.9 x 81.3 mm, 112 parts, among them IC1 BQ25303JRTER, J2 Conn_01x01_Pin, J3 Conn_01x01_Pin, J4 691213710002, J5 Pressure Sensor I/O, J6 Pressure Sensor I/O, J7 Pressure Sensor I/O, J8 JST_02, Q1 AO3400A, U1 ADS1115IDGSR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

Commit message: Final Rev to Send to Board house.
Parts:
- U12: footprint PWM Expander:QFN50P400X400X80-25N -> PWM_EXPANDER:RTW24_TEX
Connections:
- D1 pad 1: Net-(D1-PadA) -> (no net)
- D1 pad 2: Net-(IC1-STAT) -> (no net)
- U12 pad 25: GND -> (no net)
- U3 pad 12: GND -> (no net)
- U3 pad 13: GND -> (no net)
- U3 pad 14: GND -> (no net)
- U3 pad 15: GND -> (no net)
- U7 pad 2: unconnected-(U7-5V_1-Pad2) -> +5v
- U7 pad 4: Rasp_Vsupply -> unconnected-(U7-5V_2-Pad4)
Routing:
- net +5v: track 152.7 -> 177.3 mm
- net Solenoid_Driver: track 64.9 -> 62.3 mm
Other:
- outline, holes or cut-outs redrawn
